Commit message: added gate for qualification robosub

File: niot_description/models/qual_gate/urdf/qual_gate.urdf (robot description, URDF)
Before this commit: robot gate, 1 links, 0 joints
Links:
- removed link gate
- added link qual_gate, mass 18.875; collision mesh filename=package://qual_gate/meshes/qual_gate.STL; visual mesh filename=package://qual_gate/meshes/qual_gate.dae
